Commit message: Update URDF with sensor tower and GPS/LiDAR mounts
- Add 35cm sensor tower (center-mounted cylinder)
- GPS module link at base level (physical LG580P board location)
- GPS reference frame at tower top (antenna midpoint for RTK baseline)
- LiDAR frame at tower top (SLAMTEC Aurora)
- Dual antenna configuration: ±10cm Y, midpoint for position measurement
- Proper TF hierarchy: base_link → sensor_tower → gps_link/laser_frame

This represents the actual hardware configuration with GPS board
at base and antennas (±10cm Y) at tower top for RTK positioning.

File: qwacr_ws/src/qwacr_build/urdf/qwacr.urdf.xacro (robot description, xacro)
@@ -162,4 +162,99 @@
     <material>Gazebo/Purple</material>
   </gazebo>
+  <!-- Sensor Tower (35cm tall) -->
+  <link name="sensor_tower">
+    <visual>
+      <origin xyz="0 0 0.175" rpy="0 0 0"/>
+      <geometry>
+        <cylinder radius="0.025" length="0.35"/>
+      </geometry>
+      <material name="silver">
+        <color rgba="0.75 0.75 0.75 1"/>
+      </material>
+    </visual>
+    <collision>
+      <origin xyz="0 0 0.175" rpy="0 0 0"/>
+      <geometry>
+        <cylinder radius="0.025" length="0.35"/>
+      </geometry>
+    </collision>
+    <inertial>
+      <mass value="0.2"/>
+      <inertia ixx="0.0001" ixy="0.0" ixz="0.0" iyy="0.0001" iyz="0.0" izz="0.00005"/>
+    </inertial>
+  </link>
+  <joint name="base_to_sensor_tower" type="fixed">
+    <parent link="base_link"/>
+    <child link="sensor_tower"/>
+    <origin xyz="0.0 0.0 0.1" rpy="0 0 0"/>
+  </joint>
+  <!-- GPS Module (LG580P board at base level) -->
+  <link name="gps_module">
+    <visual>
+      <origin xyz="0 0 0" rpy="0 0 0"/>
+      <geometry>
+        <box size="0.08 0.06 0.02"/>
+      </geometry>
+      <material name="black">
+        <color rgba="0 0 0 1"/>
+      </material>
+    </visual>
+    <collision>
+      <origin xyz="0 0 0" rpy="0 0 0"/>
+      <geometry>
+        <box size="0.08 0.06 0.02"/>
+      </geometry>
+    </collision>
+    <inertial>
+      <mass value="0.15"/>
+      <inertia ixx="0.00002" ixy="0.0" ixz="0.0" iyy="0.00003" iyz="0.0" izz="0.00002"/>
+    </inertial>
+  </link>
+  <joint name="base_to_gps_module" type="fixed">
+    <parent link="base_link"/>
+    <child link="gps_module"/>
+    <origin xyz="-0.1 0.0 0.11" rpy="0 0 0"/>
+  </joint>
+  <!-- GPS Reference Frame (antenna midpoint at tower top) -->
+  <!-- Dual antennas at ±10cm Y, midpoint defines position measurement -->
+  <!-- Frame for GPS driver to publish position and heading -->
+  <link name="gps_link">
+    <inertial>
+      <mass value="0.001"/>
+      <inertia ixx="0.000001" ixy="0.0" ixz="0.0" iyy="0.000001" iyz="0.0" izz="0.000001"/>
+    </inertial>
+  </link>
+  <joint name="tower_to_gps" type="fixed">
+    <parent link="sensor_tower"/>
+    <child link="gps_link"/>
+    <origin xyz="0.0 0.0 0.35" rpy="0 0 0"/>
+  </joint>
+  <!-- LiDAR Sensor Link (SLAMTEC Aurora, mounted at top of tower) -->
+  <link name="laser_frame">
+    <visual>
+      <origin xyz="0 0 0" rpy="0 0 0"/>
+      <geometry>
+        <cylinder radius="0.04" length="0.025"/>
+      </geometry>
+      <material name="darkgrey">
+        <color rgba="0.2 0.2 0.2 1"/>
+      </material>
+    </visual>
+    <collision>
+      <origin xyz="0 0 0" rpy="0 0 0"/>
+      <geometry>
+        <cylinder radius="0.04" length="0.025"/>
+      </geometry>
+    </collision>
+    <inertial>
+      <mass value="0.225"/>
+      <inertia ixx="0.0001" ixy="0.0" ixz="0.0" iyy="0.0001" iyz="0.0" izz="0.0001"/>
+    </inertial>
+  </link>
+  <joint name="tower_to_laser" type="fixed">
+    <parent link="sensor_tower"/>
+    <child link="laser_frame"/>
+    <origin xyz="0.0 0.0 0.35" rpy="0 0 0"/>
+  </joint>
   <!-- ros2_control: use hardware plugin with serial simulator for development -->
   <xacro:unless value="$(arg use_gazebo)">

Commit message: Update comms, navigation, and hardware tests

File: qwacr_ws/src/qwacr_build/urdf/qwacr.urdf.xacro (robot description, xacro)
@@ -8,7 +8,7 @@
   <link name="base_link">
     <visual>
-      <origin xyz="0 0 .1" rpy="0 0 0"/>
-      <geometry>
-        <box size=".45 .3 .2"/>
+      <origin xyz="0 0 0" rpy="0 0 0"/>
+      <geometry>
+        <box size="0.8382 0.438 0.2413"/>
       </geometry>
       <material name="blue">
@@ -17,7 +17,7 @@
     </visual>
     <collision>
-      <origin xyz="0 0 .1" rpy="0 0 0"/>
-      <geometry>
-        <box size=".45 .3 .2"/>
+      <origin xyz="0 0 0" rpy="0 0 0"/>
+      <geometry>
+        <box size="0.8382 0.438 0.2413"/>
       </geometry>
     </collision>
@@ -34,6 +34,6 @@
     <parent link="base_link"/>
     <child link="front_left_wheel_link"/>
-    <origin xyz="0.18 0.19 -0.02" rpy="0 0 0"/>
-     <axis xyz="0 1 0"/>
+    <origin xyz="0.3175 0.308 -0.0699" rpy="0 0 0"/>
+     <axis xyz="0 -1 0"/>
     <limit effort="6.2" velocity="104"/>
     <dynamics damping=".0001" friction="0.001"/>
@@ -43,5 +43,5 @@
       <origin xyz="0 0 0" rpy="1.5708 0 0"/>
       <geometry>
-        <cylinder radius="0.165" length="0.06"/>
+        <cylinder radius="0.1651" length="0.1143"/>
       </geometry>
       <material name="red">
@@ -52,5 +52,5 @@
       <origin xyz="0 0 0" rpy="1.5708 0 0"/>
       <geometry>
-        <cylinder radius="0.165" length="0.06"/>
+        <cylinder radius="0.1651" length="0.1143"/>
       </geometry>
     </collision>
@@ -62,4 +62,8 @@
   <gazebo reference="front_left_wheel_link">
     <material>Gazebo/Red</material>
+    <mu1>1.0</mu1>
+    <mu2>0.5</mu2>
+    <slip1>0.5</slip1>
+    <slip2>0.0</slip2>
   </gazebo>
   <!-- Front right wheel -->
@@ -67,5 +71,5 @@
     <parent link="base_link"/>
     <child link="front_right_wheel_link"/>
-    <origin xyz="0.18 -0.19 -0.02" rpy="0 0 0"/>
+    <origin xyz="0.3175 -0.308 -0.0699" rpy="0 0 0"/>
     <axis xyz="0 1 0"/>
     <limit effort="6.2" velocity="104"/>
@@ -76,5 +80,5 @@
       <origin xyz="0 0 0" rpy="1.5708 0 0"/>
       <geometry>
-        <cylinder radius="0.165" length="0.06"/>
+        <cylinder radius="0.1651" length="0.1143"/>
       </geometry>
       <material name="green">
@@ -85,5 +89,5 @@
       <origin xyz="0 0 0" rpy="1.5708 0 0"/>
       <geometry>
-        <cylinder radius="0.165" length="0.06"/>
+        <cylinder radius="0.1651" length="0.1143"/>
       </geometry>
     </collision>
@@ -95,4 +99,8 @@
   <gazebo reference="front_right_wheel_link">
     <material>Gazebo/Green</material>
+    <mu1>1.0</mu1>
+    <mu2>0.5</mu2>
+    <slip1>0.5</slip1>
+    <slip2>0.0</slip2>
   </gazebo>
   <!-- Back left wheel -->
@@ -100,6 +108,6 @@
     <parent link="base_link"/>
     <child link="back_left_wheel_link"/>
-    <origin xyz="-0.18 0.19 -0.02" rpy="0 0 0"/>
-     <axis xyz="0 1 0"/>
+    <origin xyz="-0.3175 0.308 -0.0699" rpy="0 0 0"/>
+     <axis xyz="0 -1 0"/>
     <limit effort="6.2" velocity="104"/>
     <dynamics damping=".0001" friction="0.001"/>
@@ -109,5 +117,5 @@
       <origin xyz="0 0 0" rpy="1.5708 0 0"/>
       <geometry>
-        <cylinder radius="0.165" length="0.06"/>
+        <cylinder radius="0.1651" length="0.1143"/>
       </geometry>
       <material name="yellow">
@@ -118,5 +126,5 @@
       <origin xyz="0 0 0" rpy="1.5708 0 0"/>
       <geometry>
-        <cylinder radius="0.165" length="0.06"/>
+        <cylinder radius="0.1651" length="0.1143"/>
       </geometry>
     </collision>
@@ -128,4 +136,8 @@
   <gazebo reference="back_left_wheel_link">
     <material>Gazebo/Yellow</material>
+    <mu1>1.0</mu1>
+    <mu2>0.5</mu2>
+    <slip1>0.5</slip1>
+    <slip2>0.0</slip2>
   </gazebo>
   <!-- Back right wheel -->
@@ -133,5 +145,5 @@
     <parent link="base_link"/>
     <child link="back_right_wheel_link"/>
-    <origin xyz="-0.18 -0.19 -0.02" rpy="0 0 0"/>
+    <origin xyz="-0.3175 -0.308 -0.0699" rpy="0 0 0"/>
     <axis xyz="0 1 0"/>
     <limit effort="6.2" velocity="104"/>
@@ -142,5 +154,5 @@
       <origin xyz="0 0 0" rpy="1.5708 0 0"/>
       <geometry>
-        <cylinder radius="0.165" length="0.06"/>
+        <cylinder radius="0.1651" length="0.1143"/>
       </geometry>
       <material name="purple">
@@ -151,5 +163,5 @@
       <origin xyz="0 0 0" rpy="1.5708 0 0"/>
       <geometry>
-        <cylinder radius="0.165" length="0.06"/>
+        <cylinder radius="0.1651" length="0.1143"/>
       </geometry>
     </collision>
@@ -161,4 +173,8 @@
   <gazebo reference="back_right_wheel_link">
     <material>Gazebo/Purple</material>
+    <mu1>1.0</mu1>
+    <mu2>0.5</mu2>
+    <slip1>0.5</slip1>
+    <slip2>0.0</slip2>
   </gazebo>
   <!-- Sensor Tower (35cm tall) -->
@@ -257,4 +273,124 @@
     <origin xyz="0.0 0.0 0.35" rpy="0 0 0"/>
   </joint>
+  <!-- Gazebo Sensor Plugins (only in simulation mode) -->
+  <xacro:if value="$(arg use_gazebo)">
+    <!-- LiDAR Sensor Plugin -->
+    <gazebo reference="laser_frame">
+      <sensor name="laser_scanner" type="gpu_lidar">
+        <topic>scan</topic>
+        <update_rate>10</update_rate>
+        <lidar>
+          <scan>
+            <horizontal>
+              <samples>360</samples>
+              <resolution>1</resolution>
+              <min_angle>-3.14159</min_angle>
+              <max_angle>3.14159</max_angle>
+            </horizontal>
+          </scan>
+          <range>
+            <min>0.12</min>
+            <max>12.0</max>
+            <resolution>0.01</resolution>
+          </range>
+          <noise>
+            <type>gaussian</type>
+            <mean>0.0</mean>
+            <stddev>0.01</stddev>
+          </noise>
+        </lidar>
+        <always_on>1</always_on>
+        <visualize>true</visualize>
+      </sensor>
+    </gazebo>
+    <!-- GPS Sensor Plugin -->
+    <gazebo reference="gps_link">
+      <sensor name="gps_sensor" type="navsat">
+        <topic>gps/fix</topic>
+        <update_rate>5</update_rate>
+        <always_on>1</always_on>
+        <navsat>
+          <position_sensing>
+            <horizontal>
+              <noise type="gaussian">
+                <mean>0.0</mean>
+                <stddev>1.0</stddev>
+              </noise>
+            </horizontal>
+            <vertical>
+              <noise type="gaussian">
+                <mean>0.0</mean>
+                <stddev>2.0</stddev>
+              </noise>
+            </vertical>
+          </position_sensing>
+          <velocity_sensing>
+            <horizontal>
+              <noise type="gaussian">
+                <mean>0.0</mean>
+                <stddev>0.1</stddev>
+              </noise>
+            </horizontal>
+            <vertical>
+              <noise type="gaussian">
+                <mean>0.0</mean>
+                <stddev>0.1</stddev>
+              </noise>
+            </vertical>
+          </velocity_sensing>
+        </navsat>
+      </sensor>
+    </gazebo>
+    <!-- IMU Sensor Plugin -->
+    <gazebo reference="base_link">
+      <sensor name="imu_sensor" type="imu">
+        <topic>imu/data</topic>
+        <update_rate>50</update_rate>
+        <always_on>1</always_on>
+        <imu>
+          <angular_velocity>
+            <x>
+              <noise type="gaussian">
+                <mean>0.0</mean>
+                <stddev>0.01</stddev>
+              </noise>
+            </x>
+            <y>
+              <noise type="gaussian">
+                <mean>0.0</mean>
+                <stddev>0.01</stddev>
+              </noise>
+            </y>
+            <z>
+              <noise type="gaussian">
+                <mean>0.0</mean>
+                <stddev>0.01</stddev>
+              </noise>
+            </z>
+          </angular_velocity>
+          <linear_acceleration>
+            <x>
+              <noise type="gaussian">
+                <mean>0.0</mean>
+                <stddev>0.05</stddev>
+              </noise>
+            </x>
+            <y>
+              <noise type="gaussian">
+                <mean>0.0</mean>
+                <stddev>0.05</stddev>
+              </noise>
+            </y>
+            <z>
+              <noise type="gaussian">
+                <mean>0.0</mean>
+                <stddev>0.05</stddev>
+              </noise>
+            </z>
+          </linear_acceleration>
+        </imu>
+      </sensor>
+    </gazebo>
+  </xacro:if>
   <!-- ros2_control: use hardware plugin with serial simulator for development -->
   <xacro:unless value="$(arg use_gazebo)">
@@ -287,37 +423,35 @@
     </ros2_control>
   </xacro:unless>
-  <!-- Gazebo simulation mode: use Gazebo physics directly -->
-  <xacro:if value="$(arg use_gazebo)">
-    <ros2_control name="GazeboSystem" type="system">
-      <hardware>
-        <plugin>gz_ros2_control/GazeboSimSystem</plugin>
-      </hardware>
-      <joint name="base_to_front_left_wheel">
-        <command_interface name="velocity"/>
-        <state_interface name="velocity"/>
-        <state_interface name="position"/>
-      </joint>
-      <joint name="base_to_front_right_wheel">
-        <command_interface name="velocity"/>
-        <state_interface name="velocity"/>
-        <state_interface name="position"/>
-      </joint>
-      <joint name="base_to_back_left_wheel">
-        <command_interface name="velocity"/>
-        <state_interface name="velocity"/>
-        <state_interface name="position"/>
-      </joint>
-      <joint name="base_to_back_right_wheel">
-        <command_interface name="velocity"/>
-        <state_interface name="velocity"/>
-        <state_interface name="position"/>
-      </joint>
-    </ros2_control>
-  </xacro:if>
-  <!-- Gazebo plugin to bridge ros2_control to Gazebo physics -->
+  <!-- Gazebo simulation mode: use built-in differential drive plugin (simpler, more stable) -->
   <xacro:if value="$(arg use_gazebo)">
     <gazebo>
-      <plugin filename="libgz_ros2_control-system.so" name="gz_ros2_control::GazeboSimROS2ControlPlugin">
-        <parameters>$(find qwacr_build)/config/diff_drive_controller.yaml</parameters>
+      <plugin filename="gz-sim-diff-drive-system" name="gz::sim::systems::DiffDrive">
+        <left_joint>base_to_front_left_wheel</left_joint>
+        <left_joint>base_to_back_left_wheel</left_joint>
+        <right_joint>base_to_front_right_wheel</right_joint>
+        <right_joint>base_to_back_right_wheel</right_joint>
+        <wheel_separation>0.38</wheel_separation>
+        <wheel_radius>0.165</wheel_radius>
+        <odom_publish_frequency>50</odom_publish_frequency>
+        <max_linear_acceleration>1.0</max_linear_acceleration>
+        <min_linear_acceleration>-1.0</min_linear_acceleration>
+        <max_angular_acceleration>2.0</max_angular_acceleration>
+        <min_angular_acceleration>-2.0</min_angular_acceleration>
+        <max_linear_velocity>1.5</max_linear_velocity>
+        <min_linear_velocity>-1.5</min_linear_velocity>
+        <max_angular_velocity>3.0</max_angular_velocity>
+        <min_angular_velocity>-3.0</min_angular_velocity>
+        <topic>cmd_vel</topic>
+        <odom_topic>odom</odom_topic>
+        <tf_topic>tf</tf_topic>
+        <frame_id>odom</frame_id>
+        <child_frame_id>base_link</child_frame_id>
+        <robot_base_frame>base_link</robot_base_frame>
+      </plugin>
+      <plugin filename="gz-sim-joint-state-publisher-system" name="gz::sim::systems::JointStatePublisher">
+        <joint_name>base_to_front_left_wheel</joint_name>
+        <joint_name>base_to_front_right_wheel</joint_name>
+        <joint_name>base_to_back_left_wheel</joint_name>
+        <joint_name>base_to_back_right_wheel</joint_name>
       </plugin>
     </gazebo>

Commit message: Update arduino firmware, diff drive control, comms, gps driver, and nav launch files

File: qwacr_ws/src/qwacr_build/urdf/qwacr.urdf.xacro (robot description, xacro)
@@ -35,5 +35,5 @@
     <child link="front_left_wheel_link"/>
     <origin xyz="0.3175 0.308 -0.0699" rpy="0 0 0"/>
-     <axis xyz="0 -1 0"/>
+     <axis xyz="0 1 0"/>
     <limit effort="6.2" velocity="104"/>
     <dynamics damping=".0001" friction="0.001"/>
@@ -109,5 +109,5 @@
     <child link="back_left_wheel_link"/>
     <origin xyz="-0.3175 0.308 -0.0699" rpy="0 0 0"/>
-     <axis xyz="0 -1 0"/>
+     <axis xyz="0 1 0"/>
     <limit effort="6.2" velocity="104"/>
     <dynamics damping=".0001" friction="0.001"/>
